Commit message: added color param

File: nuturtle_description/urdf/turtlebot3_burger.urdf.xacro (robot description, xacro)
@@ -1,4 +1,6 @@
 <?xml version="1.0" ?>
 <robot name="turtlebot3_burger" xmlns:xacro="http://ros.org/wiki/xacro">
+<xacro:include filename="$(find nuturtle_description)/urdf/turtlebot3_burger.gazebo.xacro"/>
+<xacro:arg name="color" default="purple"/>
 <xacro:property name="yaml_file" value="$(find nuturtle_description)/config/diff_params.yaml" />
 <xacro:property name="config" value="${xacro.load_yaml(yaml_file)['nuturtle_description']['ros__parameters']}" />
@@ -9,7 +11,16 @@
 <xacro:property name="encoder_ticks_per_rad"  value="${config['encoder_ticks_per_rad']}" />
 <xacro:property name="collision_radius"  value="${config['collision_radius']}" />
-<xacro:arg name="color" default="purple"/>
-  <xacro:include filename="$(find nuturtle_description)/urdf/common_properties.xacro"/>
-  <xacro:include filename="$(find nuturtle_description)/urdf/turtlebot3_burger.gazebo.xacro"/>
+  <material name="purple">
+    <color rgba="0.3 0.16 0.52 1.0"/>
+  </material>
+  <material name="red">
+    <color rgba="0.8 0 0 1.0"/>
+  </material>
+  <material name="green">
+    <color rgba="0 0.8 0 1.0"/>
+  </material>
+  <material name="blue">
+    <color rgba="0 0 0.8 1.0"/>
+  </material>
   <link name="base_footprint"/>
   <joint name="base_joint" type="fixed">
@@ -24,5 +35,5 @@
         <mesh filename="package://nuturtle_description/meshes/burger_base.stl" scale="0.001 0.001 0.001"/>
       </geometry>
-      <material name="light_black"/>
+      <material name="$(arg color)"/>
     </visual>
     <collision>
@@ -52,5 +63,5 @@
         <mesh filename="package://nuturtle_description/meshes/left_tire.stl" scale="0.001 0.001 0.001"/>
       </geometry>
-      <material name="dark"/>
+      <material name="$(arg color)"/>
     </visual>
     <collision>
@@ -80,5 +91,5 @@
         <mesh filename="package://nuturtle_description/meshes/right_tire.stl" scale="0.001 0.001 0.001"/>
       </geometry>
-      <material name="dark"/>
+      <material name="$(arg color)"/>
     </visual>
     <collision>
@@ -133,5 +144,5 @@
         <mesh filename="package://nuturtle_description/meshes/lds.stl" scale="0.001 0.001 0.001"/>
       </geometry>
-      <material name="dark"/>
+      <material name="$(arg color)"/>
     </visual>
     <collision>

Commit message: finished task a4, can load all robot colors in rviz

File: nuturtle_description/urdf/turtlebot3_burger.urdf.xacro (robot description, xacro)
@@ -22,4 +22,7 @@
   <material name="blue">
     <color rgba="0 0 0.8 1.0"/>
+  </material>
+  <material name="dark">
+    <color rgba="0.1 0.1 0.1 1.0"/>
   </material>
   <link name="base_footprint"/>
@@ -63,5 +66,5 @@
         <mesh filename="package://nuturtle_description/meshes/left_tire.stl" scale="0.001 0.001 0.001"/>
       </geometry>
-      <material name="$(arg color)"/>
+      <material name="dark"/>
     </visual>
     <collision>
@@ -91,5 +94,5 @@
         <mesh filename="package://nuturtle_description/meshes/right_tire.stl" scale="0.001 0.001 0.001"/>
       </geometry>
-      <material name="$(arg color)"/>
+      <material name="dark"/>
     </visual>
     <collision>
@@ -144,5 +147,5 @@
         <mesh filename="package://nuturtle_description/meshes/lds.stl" scale="0.001 0.001 0.001"/>
       </geometry>
-      <material name="$(arg color)"/>
+      <material name="dark"/>
     </visual>
     <collision>

Commit message: added all functionality to turtle_control launchfile except rviz

File: nuturtle_description/urdf/turtlebot3_burger.urdf.xacro (robot description, xacro)
@@ -4,5 +4,5 @@
 <xacro:arg name="color" default="purple"/>
 <xacro:property name="yaml_file" value="$(find nuturtle_description)/config/diff_params.yaml" />
-<xacro:property name="config" value="${xacro.load_yaml(yaml_file)['nuturtle_description']['ros__parameters']}" />
+<xacro:property name="config" value="${xacro.load_yaml(yaml_file)['/**']['ros__parameters']}" />
 <xacro:property name="wheel_radius"  value="${config['wheel_radius']}" />
 <xacro:property name="track_width"  value="${config['track_width']}" />

Commit message: fixed speed issues, fixed RViz issues, robots display correctly now

File: nuturtle_description/urdf/turtlebot3_burger.urdf.xacro (robot description, xacro)
@@ -5,5 +5,5 @@
 <xacro:property name="yaml_file" value="$(find nuturtle_description)/config/diff_params.yaml" />
 <xacro:property name="config" value="${xacro.load_yaml(yaml_file)['/**']['ros__parameters']}" />
-<xacro:property name="wheel_radius"  value="${config['wheel_radius']}" />
+<xacro:property name="wheel_diameter"  value="${config['wheel_diameter']}" />
 <xacro:property name="track_width"  value="${config['track_width']}" />
 <xacro:property name="motor_cmd_max"  value="${config['motor_cmd_max']}" />
@@ -71,5 +71,5 @@
       <origin xyz="0 0 0" rpy="0 0 0"/>
       <geometry>
-        <cylinder length="0.018" radius="${wheel_radius/2}"/>
+        <cylinder length="0.018" radius="${wheel_diameter/2}"/>
       </geometry>
     </collision>
@@ -99,5 +99,5 @@
       <origin xyz="0 0 0" rpy="0 0 0"/>
       <geometry>
-        <cylinder length="0.018" radius="${wheel_radius/2}"/>
+        <cylinder length="0.018" radius="${wheel_diameter/2}"/>
       </geometry>
     </collision>
